File: HV_Stuff/HV_schematic.sch (EAGLE design)
At the start: 0 parts

Commit message: Made basic schematic with Arduino board included
Next step is designing PCB
Parts:
- added B2: ARDUINO_UNO_R3_SHIELDBASIC, SparkFun-Boards:ARDUINO_UNO_R3_SHIELDBASIC
- added JP1, JP2: (no value), jumper:JP4E
- added JP3, JP4, JP7, JP8: (no value), jumper:JP1E
Connections:
- new net GND: B2.GND@2, JP1.4
- new net IN1: JP3.2
- new net IN2: JP3.1
- new net IN3: JP1.2
- new net IN4: JP1.1
- new net OUT1: JP2.3, JP7.1
- new net OUT2: JP2.2, JP7.2
- new net OUT3: JP2.1, JP8.1
- new net OUT4: JP4.2, JP8.2
- new net VCC: B2.VIN, JP1.3
Other:
- note added: "facing the board (pins pointing at you)"
